File: KiCad scheme/KiCad scheme.sch (KiCad schematic (older format))
At the start: 4 parts

Commit message: scheme
Parts:
- U?: symbol Sensor_Distance:InfraRed -> KiCad-scheme-rescue:InfraRed-Sensor_Distance
Connections:
- net at ESP8266.4 (3V3): now also U?.3 (VDD), U?.~ (VCC)
- now unconnected: ESP8266.5 (+5V)
Changed lines of the file:
@@
 Wire Wire Line
 	1900 4200 1900 4450
-Wire Wire Line
-	3400 4300 1600 4300
-Wire Wire Line
-	1600 4300 1600 4450
 Connection ~ 1800 6800
 $Comp
-L Sensor_Distance:InfraRed U?
+L KiCad-scheme-rescue:InfraRed-Sensor_Distance U?
 U 1 1 604BD4C7
 P 3400 5250
@@
 Wire Wire Line
 	3100 6800 2500 6800
+Wire Wire Line
+	3400 4300 1700 4300
+Wire Wire Line
+	1700 4300 1700 4450
 $EndSCHEMATC
