File: KiCadScheme/KiCad scheme.sch (KiCad schematic (older format))
At the start: 4 parts

Commit message: final schematic
Parts:
- removed U?: InfraRed, symbol KiCad-scheme-rescue:InfraRed-Sensor_Distance
- removed U?: DS18B20, Package_TO_SOT_THT:TO-92_Inline, symbol Sensor_Temperature:DS18B20
- added D?: LED, symbol Device:LED
- added U?: Light, symbol Sensor_Motion:Light
Connections:
- net at ESP8266.29 (GND), ESP8266.6 (GND), ESP8266.7 (GND)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: now also D?.1 (K), U?.~ (VCC)
- net at ESP8266.4 (3V3): now also U?.~ (VCC)
- net at ESP8266.16 (D1/TX): now also U?.~ (VCC)
- net at ESP8266.23 (D8): now also D?.2 (A)
Changed lines of the file:
@@
-$EndComp
-$Comp
-L Sensor_Temperature:DS18B20 U?
-U 1 1 604C4234
-P 3100 5600
-F 0 "U?" H 2870 5646 50  0000 R CNN
-F 1 "DS18B20" H 2870 5555 50  0000 R CNN
-F 2 "Package_TO_SOT_THT:TO-92_Inline" H 2100 5350 50  0001 C CNN
-F 3 "http://datasheets.maximintegrated.com/en/ds/DS18B20.pdf" H 2950 5850 50  0001 C CNN
-	1    3100 5600
-	-1   0    0    -1
 $EndComp
 $Comp
@@
 	1900 4200 1900 4450
 Connection ~ 1800 6800
+Wire Wire Line
+	1700 4300 1700 4450
 $Comp
-L KiCad-scheme-rescue:InfraRed-Sensor_Distance U?
-U 1 1 604BD4C7
-P 3400 5250
-F 0 "U?" H 3729 5659 50  0000 C CNN
-F 1 "InfraRed" H 3729 5576 39  0000 C CNN
-F 2 "" H 3400 5250 50  0001 C CNN
-F 3 "" H 3400 5250 50  0001 C CNN
-	1    3400 5250
+L Device:LED D?
+U 1 1 604D96B0
+P 3900 5150
+F 0 "D?" H 3893 4895 50  0000 C CNN
+F 1 "LED" H 3893 4986 50  0000 C CNN
+F 2 "" H 3900 5150 50  0001 C CNN
+F 3 "~" H 3900 5150 50  0001 C CNN
+	1    3900 5150
+	-1   0    0    1
+$EndComp
+Wire Wire Line
+	1800 6800 2500 6800
+$Comp
+L Sensor_Motion:Light U?
+U 1 1 604DC9C1
+P 2800 5000
+F 0 "U?" H 3100 5050 50  0000 L CNN
+F 1 "Light" H 3100 4850 50  0000 L CNN
+F 2 "" H 3150 5000 50  0001 C CNN
+F 3 "" H 3150 5000 50  0001 C CNN
+	1    2800 5000
 	1    0    0    -1
 $EndComp
 Wire Wire Line
-	3400 5050 2300 5050
+	1700 4300 2750 4300
 Wire Wire Line
-	3400 4900 3100 4900
+	2750 4300 2750 5100
 Wire Wire Line
-	3100 4900 3100 5300
+	2750 5150 2500 5150
 Wire Wire Line
-	3100 5300 3400 5300
-Wire Wire Line
-	3400 5300 3400 5150
-Wire Wire Line
-	3400 4300 3400 4900
-Wire Wire Line
-	3400 5100 2500 5100
-Wire Wire Line
-	2500 5100 2500 6800
+	2500 5150 2500 6800
 Connection ~ 2500 6800
 Wire Wire Line
-	2500 6800 1800 6800
-Connection ~ 3100 5300
+	2750 5200 2450 5200
 Wire Wire Line
-	2300 5150 2800 5150
+	2450 5200 2450 4950
 Wire Wire Line
-	2800 5150 2800 5600
+	2450 4950 2300 4950
 Wire Wire Line
-	3100 5900 3100 6800
+	4050 5150 4050 6800
 Wire Wire Line
-	3100 6800 2500 6800
+	2500 6800 4050 6800
 Wire Wire Line
-	3400 4300 1700 4300
+	3750 5150 3750 5650
 Wire Wire Line
-	1700 4300 1700 4450
+	3750 5650 2300 5650
 $EndSCHEMATC
